File: EasyCT.kicad_sch (KiCad schematic)
At the start: 18 parts, among them CN1 SCT013, J1 Screw_Terminal_01x02, U1 MCP6002-xP

Commit message: feat: finish v1, send to JLCPCB
Parts:
- removed C2: 0.1μF, symbol Device:C_Polarized
- removed D3: D, symbol Device:D
- removed R4: R_Trim, symbol Device:R_Trim
- removed U1: MCP6002-xP, symbol Amplifier_Operational:MCP6002-xP
- added C1, C3, C7, C8: 100nF, Capacitor_SMD:C_0805_2012Metric, symbol Device:C
- added C2, C5: 4.7μF, Capacitor_SMD:C_0805_2012Metric, symbol Device:C
- added C4: 10nF, Capacitor_SMD:C_0805_2012Metric, symbol Device:C
- added C9: 10μF, Capacitor_SMD:C_0805_2012Metric, symbol Device:C
- added D2, D4: 1N4148, Diode_SMD:D_SOD-123, symbol Device:D
- added D5, D6, D7: 1N5819W, Diode_SMD:D_SOD-323, symbol Device:D
- added H1, H2, H3: MountingHole, MountingHole:MountingHole_3.2mm_M3, symbol Mechanical:MountingHole
- added J2: Screw_Terminal_01x07, EasyCT_Vendored:CONN-TH_XY308-2.54-7P, symbol Connector:Screw_Terminal_01x07
- added JP1, JP2: SolderJumper_2_Open, Jumper:SolderJumper-2_P1.3mm_Open_TrianglePad1.0x1.5mm, symbol Jumper:SolderJumper_2_Open
- added Q1: IRLML0040TRPbF, Package_TO_SOT_SMD:SOT-23, symbol Simulation_SPICE:NMOS
- added R10: 1M, Resistor_SMD:R_0805_2012Metric, symbol Device:R
- added R11: 1K, Resistor_SMD:R_0805_2012Metric, symbol Device:R
- added R4: R, Resistor_THT:R_Axial_DIN0207_L6.3mm_D2.5mm_P7.62mm_Horizontal, symbol Device:R
- added R9: 47K, Resistor_SMD:R_0805_2012Metric, symbol Device:R
- added RV1: 200K, Potentiometer_THT:Potentiometer_Bourns_3296W_Vertical, symbol Device:R_Potentiometer_Trim
- added TP1: TestPoint_2Pole, TestPoint:TestPoint_2Pads_Pitch5.08mm_Drill1.3mm, symbol Connector:TestPoint_2Pole
- added U1: RT9193-30GB, EasyCT_Vendored:SOT-23-5_L3.0-W1.7-P0.95-LS2.8-BR, symbol EasyCT_Vendored:RT9193-30GB
- added U2, U3: LMV321, Package_TO_SOT_SMD:SOT-23-5, symbol Amplifier_Operational:LMV321
- C6: renamed from C1; footprint (none) -> Capacitor_SMD:C_0805_2012Metric
- D1: value D -> 1N4148; footprint (none) -> Diode_SMD:D_SOD-123
- D3: renamed from D2; value D -> 1N4148; footprint (none) -> Diode_SMD:D_SOD-123
- J1: footprint (none) -> EasyCT_Vendored:CONN-TH_XY308-2.54-2P
- R1, R2, R3, R5, R6: footprint (none) -> Resistor_THT:R_Axial_DIN0207_L6.3mm_D2.5mm_P7.62mm_Horizontal
- R7, R8: value R -> 47K; footprint (none) -> Resistor_SMD:R_0805_2012Metric
Connections:
- net OUT1 is gone; now on an unnamed net: R6.1
- net GND: now also J1.2 (Pin_2), R8.1, C1.1, C2.1, C3.1, C5.1, C7.2, C8.2, C9.2, D2.1 (K), D4.2 (A), D5.2 (A), J2.1 (Pin_1), JP2.1 (A), Q1.3 (S), R10.2, R4.2, RV1.3, TP1.1, U1.2 (GND), U2.2 (V-), U3.2 (V-); no longer D1.1 (K), D3.2 (A), J1.1 (Pin_1), R3.1, R7.1
- net VCC: now also C1.2, C2.2, C7.1, J2.2 (Pin_2), U1.1 (VIN), U1.3 (EN), U2.5 (V+); no longer R1.1, R5.2, R8.2
- net at R1.2, R2.1: now also R3.2, R5.2, JP1.1 (A), JP2.2 (B), R4.1; no longer C6.1
- net at R7.2: now also D5.1 (K), U3.1 (+); no longer R8.1
- net R_B_IN: now reaches R5.1
- net R_B_IN: now also C6.2, CN1.4 (+), D1.2 (A), D3.1 (K), J1.1 (Pin_1), L1.2 (+), L2.2 (+), R1.1, R3.1, JP1.2 (B)
- removed net SENSE: C6.2, CN1.4 (+), D1.2 (A), D3.1 (K), J1.2 (Pin_2), L1.2 (+), L2.2 (+)
- new net: D3.2 (A), D4.1 (K)
- new net: C4.2, U1.4 (BP)
- new net: R8.2, R9.1, U3.3 (-)
- new net: Q1.2 (G), R11.2
- new net: D6.2 (A), U3.4
- new net: D1.1 (K), D2.2 (A)
- new net +3V0: C3.2, C4.1, C5.2, C8.1, RV1.1, U1.5 (VOUT), U3.5 (V+)
- new net OUT_ANALOG: C9.1, D6.1 (K), J2.4 (Pin_4), R10.1, R9.2, U2.1 (+)
- new net OUT_DIGITAL: J2.3 (Pin_3), R11.1, U2.4
- new net SW_GND: D7.2 (A), J2.5 (Pin_5), Q1.1 (D)
- new net SW_VCC: D7.1 (K), J2.6 (Pin_6), J2.7 (Pin_7)
- new net S_OUT: C6.1, R7.1
- new net V_TRIGGER: RV1.2, TP1.2, U2.3 (-)
Other:
- note added: "Inspired by: https://github.com/DFRobot/DFRobot_AnalogACurrentSensor (LGPL v3)"
- note removed: "Trim to zero op-amp output when I_in = 0A"
- company: (none) -> Jeppe Klitgaard
- title: (none) -> EasyCT
- moved on the sheet: C6, D1, D3
